Commit message: after adding legs but i will work on changing joints of rotations

File: spidy/urdf/spidy_desc.urdf (robot description, URDF)
Before this commit: robot myfirst, 5 links, 4 joints
Links:
- added link front_bo2la_2; visual cylinder length=0.3 radius=0.1
- added link front_leg; visual box size=0.1 0.6 0.3
- added link front_leg_2; visual box size=0.1 0.4 0.1
- added link left_bo2la_2; visual cylinder length=0.3 radius=0.1
- added link left_leg; visual box size=0.1 0.6 0.3
- added link left_leg_2; visual box size=0.1 0.4 0.1
- added link right_bo2la_2; visual cylinder length=0.3 radius=0.1
- added link right_leg; visual box size=0.1 0.6 0.3
- added link right_leg_2; visual box size=0.1 0.4 0.1
Joints:
- added joint front_bo2la_2_to_front_leg_2: type continuous, parent front_bo2la_2, child front_leg_2, origin xyz=0 0 -0.3 rpy=0 0 0
- added joint front_bo2la_to_front_leg: type continuous, parent front_bo2la, child front_leg, origin xyz=0.4 0 0 rpy=0 0 0
- added joint front_leg_to_front_bo2la_2: type fixed, parent front_leg, child front_bo2la_2, origin xyz=0.4 0 0 rpy=0 0 0
- added joint left_bo2la_2_to_left_leg: type continuous, parent left_bo2la_2, child left_leg_2, origin xyz=0 0 -0.3 rpy=0 0 0
- added joint left_bo2la_to_left_leg: type continuous, parent left_bo2la, child left_leg, origin xyz=0 0.4 0 rpy=0 0 0
- added joint left_leg_to_left_bo2la_2: type fixed, parent left_leg, child left_bo2la_2, origin xyz=0 0.4 0 rpy=0 0 0
- added joint right_bo2la_2_to_right_leg_2: type continuous, parent right_bo2la_2, child right_leg_2, origin xyz=0 0 -0.3 rpy=0 0 0
- added joint right_bo2la_to_right_leg: type continuous, parent right_bo2la, child right_leg, origin xyz=0 -0.4 0 rpy=0 0 0
- added joint right_leg_to_right_bo2la_2: type fixed, parent right_leg, child right_bo2la_2, origin xyz=0 -0.4 0 rpy=0 0 0

Commit message: after resolving joints issue

File: spidy/urdf/spidy_desc.urdf (robot description, URDF)
Before this commit: robot myfirst, 14 links, 13 joints
Links:
- added link back_bo2la_2; visual cylinder length=0.3 radius=0.1
- added link back_leg; visual box size=0.1 0.6 0.3
- added link back_leg_2; visual box size=0.1 0.4 0.1
Joints:
- added joint back_bo2la_2_to_back_leg_2: type continuous, parent back_bo2la_2, child back_leg_2, origin xyz=0 0 0 rpy=0 0 0, axis 0 1 0
- added joint back_bo2la_to_back_leg: type continuous, parent back_bo2la, child back_leg, origin xyz=0 0 0 rpy=0 0 0, axis 0 0 1
- added joint back_leg_to_back_bo2la_2: type fixed, parent back_leg, child back_bo2la_2, origin xyz=-0.6 0 0 rpy=0 0 0
- joint front_bo2la_2_to_front_leg_2: axis (none) -> 0 1 0; origin xyz=0 0 -0.3 rpy=0 0 0 -> xyz=0 0 0 rpy=0 0 0
- joint front_bo2la_to_front_leg: axis (none) -> 0 0 1; origin xyz=0.4 0 0 rpy=0 0 0 -> xyz=0 0 0 rpy=0 0 0
- joint front_leg_to_front_bo2la_2: origin xyz=0.4 0 0 rpy=0 0 0 -> xyz=0.6 0 0 rpy=0 0 0
- joint left_bo2la_2_to_left_leg: origin xyz=0 0 -0.3 rpy=0 0 0 -> xyz=0 0 0 rpy=0 0 0
- joint left_bo2la_to_left_leg: axis (none) -> 0 0 1; origin xyz=0 0.4 0 rpy=0 0 0 -> xyz=0 0 0 rpy=0 0 0
- joint left_leg_to_left_bo2la_2: origin xyz=0 0.4 0 rpy=0 0 0 -> xyz=0 0.6 0 rpy=0 0 0
- joint right_bo2la_2_to_right_leg_2: origin xyz=0 0 -0.3 rpy=0 0 0 -> xyz=0 0 0 rpy=0 0 0
- joint right_bo2la_to_right_leg: axis (none) -> 0 0 1; origin xyz=0 -0.4 0 rpy=0 0 0 -> xyz=0 0 0 rpy=0 0 0
- joint right_leg_to_right_bo2la_2: origin xyz=0 -0.4 0 rpy=0 0 0 -> xyz=0 -0.6 0 rpy=0 0 0

Commit message: after spawning in gazebo

File: spidy/urdf/spidy_desc.urdf (robot description, URDF)
Before this commit: robot myfirst, 17 links, 16 joints
Links:
- link back_bo2la: mass None -> 10; geometry collision cylinder length=0.3 radius=0.1; visual cylinder length=0.3 radius=0.1
- link back_bo2la_2: mass None -> 10; geometry collision cylinder length=0.3 radius=0.1; visual cylinder length=0.3 radius=0.1
- link back_leg: mass None -> 10; geometry collision box size=0.1 0.6 0.3; visual box size=0.1 0.6 0.3
- link back_leg_2: mass None -> 10; geometry collision box size=0.1 0.4 0.1; visual box size=0.1 0.4 0.1
- link base_link: mass None -> 10; geometry collision cylinder length=0.3 radius=0.5; visual cylinder length=0.3 radius=0.5
- link front_bo2la: mass None -> 10; geometry collision cylinder length=0.3 radius=0.1; visual cylinder length=0.3 radius=0.1
- link front_bo2la_2: mass None -> 10; geometry collision cylinder length=0.3 radius=0.1; visual cylinder length=0.3 radius=0.1
- link front_leg: mass None -> 10; geometry collision box size=0.1 0.6 0.3; visual box size=0.1 0.6 0.3
- link front_leg_2: mass None -> 10; geometry collision box size=0.1 0.4 0.1; visual box size=0.1 0.4 0.1
- link left_bo2la: mass None -> 10; geometry collision cylinder length=0.3 radius=0.1; visual cylinder length=0.3 radius=0.1
- link left_bo2la_2: mass None -> 10; geometry collision cylinder length=0.3 radius=0.1; visual cylinder length=0.3 radius=0.1
- link left_leg: mass None -> 10; geometry collision box size=0.1 0.6 0.3; visual box size=0.1 0.6 0.3
- link left_leg_2: mass None -> 10; geometry collision box size=0.1 0.4 0.1; visual box size=0.1 0.4 0.1
- link right_bo2la: mass None -> 10; geometry collision cylinder length=0.3 radius=0.1; visual cylinder length=0.3 radius=0.1
- link right_bo2la_2: mass None -> 10; geometry collision cylinder length=0.3 radius=0.1; visual cylinder length=0.3 radius=0.1
- link right_leg: mass None -> 10; geometry collision box size=0.1 0.6 0.3; visual box size=0.1 0.6 0.3
- link right_leg_2: mass None -> 10; geometry collision box size=0.1 0.4 0.1; visual box size=0.1 0.4 0.1

Commit message: after adding the python script

File: spidy/urdf/spidy_desc.urdf (robot description, URDF)
Before this commit: robot myfirst, 17 links, 16 joints
Joints:
- removed joint left_bo2la_2_to_left_leg
- added joint left_bo2la_2_to_left_leg_2: type continuous, parent left_bo2la_2, child left_leg_2, origin xyz=0 0 0 rpy=0 0 0

Commit message: camera_addtion

File: spidy/urdf/spidy_desc.urdf (robot description, URDF)
Before this commit: robot myfirst, 17 links, 16 joints
Links:
- added link camera, mass 0.1; collision box size=0.05 0.05 0.05; visual box size=0.05 0.05 0.05
Joints:
- added joint camera_joint: type fixed, parent left_leg, child camera, origin xyz=0 0 0.175 rpy=0 0 0, axis 0 1 0
